Commit message: modify to support servobot

File: servobot/servobot.urdf (robot description, URDF)
Before this commit: robot robot, 13 links, 12 joints
Links:
- link botlegasm: geometry collision mesh filename=botleg.stl; collision mesh filename=servo.stl
- link botlegasm_2: geometry collision mesh filename=botleg.stl; collision mesh filename=servo.stl
- link botlegasm_3: geometry collision mesh filename=botleg.stl; collision mesh filename=servo.stl
- link botlegasm_4: geometry collision mesh filename=botleg.stl; collision mesh filename=servo.stl
- link hipsubasm: geometry collision mesh filename=hipjoint.stl; collision mesh filename=servo.stl
- link hipsubasm_2: geometry collision mesh filename=hipjoint.stl; collision mesh filename=servo.stl
- link mainbody: geometry collision mesh filename=base.stl; collision mesh filename=servo.stl
- link mirroredhipsubasm: geometry collision mesh filename=mirrorhipjoint.stl; collision mesh filename=servo.stl
- link mirroredhipsubasm_2: geometry collision mesh filename=mirrorhipjoint.stl; collision mesh filename=servo.stl
- link toplegasm: geometry collision mesh filename=servohornreplacement.stl; collision mesh filename=servohornreplacement.stl
- link toplegasm_2: geometry collision mesh filename=servohornreplacement.stl; collision mesh filename=servohornreplacement.stl
- link toplegasm_3: geometry collision mesh filename=servohornreplacement.stl; collision mesh filename=servohornreplacement.stl
- link toplegasm_4: geometry collision mesh filename=servohornreplacement.stl; collision mesh filename=servohornreplacement.stl

Commit message: Modified the train file and redesigned the reinforcement learning to give the robot a target area to move forward

File: servobot/servobot.urdf (robot description, URDF)
Before this commit: robot robot, 13 links, 12 joints
Links:
- removed link botlegasm
- removed link botlegasm_2
- removed link botlegasm_3
- removed link botlegasm_4
- removed link hipsubasm
- removed link hipsubasm_2
- removed link mirroredhipsubasm
- removed link mirroredhipsubasm_2
- removed link toplegasm
- removed link toplegasm_2
- removed link toplegasm_3
- removed link toplegasm_4
- added link leg_bl, mass 0.08; collision sphere radius=0.01; visual mesh filename=botleg.stl
- added link leg_br, mass 0.08; collision sphere radius=0.01; visual mesh filename=botleg.stl
- added link leg_fl, mass 0.08; collision sphere radius=0.01; visual mesh filename=botleg.stl
- added link leg_fr, mass 0.08; collision sphere radius=0.01; visual mesh filename=botleg.stl
- link mainbody: mass 0.493948 -> 1.5; geometry collision mesh filename=base.stl; visual mesh filename=base.stl
Joints:
- removed joint BL_BotLeg
- removed joint BL_TopLeg
- removed joint BR_BotLeg
- removed joint BR_TopLeg
- removed joint FL_BotLeg
- removed joint FL_TopLeg
- removed joint FR_BotLeg
- removed joint FR_TopLeg
- joint BL_Hip: child mirroredhipsubasm -> leg_bl; limit lower=-0.785398 upper=0.785398 effort=10 velocity=10 -> lower=-1.5708 upper=1.5708 effort=50 velocity=20
- joint BR_Hip: child hipsubasm_2 -> leg_br; limit lower=-0.785398 upper=0.785398 effort=10 velocity=10 -> lower=-1.5708 upper=1.5708 effort=50 velocity=20
- joint FL_Hip: child mainbody -> leg_fl; limit lower=-0.785398 upper=0.785398 effort=10 velocity=10 -> lower=-1.5708 upper=1.5708 effort=50 velocity=20; parent hipsubasm -> mainbody
- joint FR_Hip: child mirroredhipsubasm_2 -> leg_fr; limit lower=-0.785398 upper=0.785398 effort=10 velocity=10 -> lower=-1.5708 upper=1.5708 effort=50 velocity=20

Commit message: established ubuntu docker container infrastructure for running things faster

File: servobot/servobot.urdf (robot description, URDF)
Before this commit: robot robot, 13 links, 12 joints
Joints:
- joint BL_BotLeg: limit lower=-3.141592653589793 upper=3.141592653589793 effort=10 velocity=10 -> lower=-3.141592653589793 upper=3.141592653589793 effort=1 velocity=1
- joint BL_Hip: limit lower=-0.785398 upper=0.785398 effort=10 velocity=10 -> lower=-0.785398 upper=0.785398 effort=1 velocity=1
- joint BL_TopLeg: limit lower=-1.5708 upper=1.5708 effort=10 velocity=10 -> lower=-1.5708 upper=1.5708 effort=1 velocity=1
- joint BR_BotLeg: limit lower=-3.141592653589793 upper=3.141592653589793 effort=10 velocity=10 -> lower=-3.141592653589793 upper=3.141592653589793 effort=1 velocity=1
- joint BR_Hip: limit lower=-0.785398 upper=0.785398 effort=10 velocity=10 -> lower=-0.785398 upper=0.785398 effort=1 velocity=1
- joint BR_TopLeg: limit lower=-1.5708 upper=1.5708 effort=10 velocity=10 -> lower=-1.5708 upper=1.5708 effort=1 velocity=1
- joint FL_BotLeg: limit lower=-3.141592653589793 upper=3.141592653589793 effort=10 velocity=10 -> lower=-3.141592653589793 upper=3.141592653589793 effort=1 velocity=1
- joint FL_Hip: limit lower=-0.785398 upper=0.785398 effort=10 velocity=10 -> lower=-0.785398 upper=0.785398 effort=1 velocity=1
- joint FL_TopLeg: limit lower=-1.5708 upper=1.5708 effort=10 velocity=10 -> lower=-1.5708 upper=1.5708 effort=1 velocity=1
- joint FR_BotLeg: limit lower=-3.141592653589793 upper=3.141592653589793 effort=10 velocity=10 -> lower=-3.141592653589793 upper=3.141592653589793 effort=1 velocity=1
- joint FR_Hip: limit lower=-0.785398 upper=0.785398 effort=10 velocity=10 -> lower=-0.785398 upper=0.785398 effort=1 velocity=1
- joint FR_TopLeg: limit lower=-1.5708 upper=1.5708 effort=10 velocity=10 -> lower=-1.5708 upper=1.5708 effort=1 velocity=1

Commit message: added full servobot

File: servobot/servobot.urdf (robot description, URDF)
Before this commit: robot servobot, 5 links, 4 joints
Joints:
- joint BL_Hip: limit lower=-1.5708 upper=1.5708 effort=50 velocity=20 -> lower=-1.5708 upper=1.5708 effort=1.8 velocity=6
- joint BR_Hip: limit lower=-1.5708 upper=1.5708 effort=50 velocity=20 -> lower=-1.5708 upper=1.5708 effort=1.8 velocity=6
- joint FL_Hip: limit lower=-1.5708 upper=1.5708 effort=50 velocity=20 -> lower=-1.5708 upper=1.5708 effort=1.8 velocity=6
- joint FR_Hip: limit lower=-1.5708 upper=1.5708 effort=50 velocity=20 -> lower=-1.5708 upper=1.5708 effort=1.8 velocity=6
