Commit message: Fixed

File: full_servobot/catbot.urdf (robot description, URDF)
Before this commit: robot catbot, 13 links, 12 joints
Joints:
- joint BL_BotLeg: limit lower=-3.141592653589793 upper=3.141592653589793 effort=10 velocity=10 -> lower=-3.141592653589793 upper=3.141592653589793 effort=1.8 velocity=6
- joint BL_Hip: limit lower=-0.785398 upper=0.785398 effort=10 velocity=10 -> lower=-0.785398 upper=0.785398 effort=1.8 velocity=6
- joint BL_TopLeg: limit lower=-1.5708 upper=1.5708 effort=10 velocity=10 -> lower=-1.5708 upper=1.5708 effort=1.8 velocity=6
- joint BR_BotLeg: limit lower=-3.141592653589793 upper=3.141592653589793 effort=10 velocity=10 -> lower=-3.141592653589793 upper=3.141592653589793 effort=1.8 velocity=6
- joint BR_Hip: limit lower=-0.785398 upper=0.785398 effort=10 velocity=10 -> lower=-0.785398 upper=0.785398 effort=1.8 velocity=6
- joint BR_TopLeg: limit lower=-1.5708 upper=1.5708 effort=10 velocity=10 -> lower=-1.5708 upper=1.5708 effort=1.8 velocity=6
- joint FL_BotLeg: limit lower=-3.141592653589793 upper=3.141592653589793 effort=10 velocity=10 -> lower=-3.141592653589793 upper=3.141592653589793 effort=1.8 velocity=6
- joint FL_Hip: limit lower=-0.785398 upper=0.785398 effort=10 velocity=10 -> lower=-0.785398 upper=0.785398 effort=1.8 velocity=6
- joint FL_TopLeg: limit lower=-1.5708 upper=1.5708 effort=10 velocity=10 -> lower=-1.5708 upper=1.5708 effort=1.8 velocity=6
- joint FR_BotLeg: limit lower=-3.141592653589793 upper=3.141592653589793 effort=10 velocity=10 -> lower=-3.141592653589793 upper=3.141592653589793 effort=1.8 velocity=6
- joint FR_Hip: limit lower=-0.785398 upper=0.785398 effort=10 velocity=10 -> lower=-0.785398 upper=0.785398 effort=1.8 velocity=6
- joint FR_TopLeg: limit lower=-1.5708 upper=1.5708 effort=10 velocity=10 -> lower=-1.5708 upper=1.5708 effort=1.8 velocity=6
