Commit message: Changed the start position and fixed a few bugs

File: simple_quadruped.urdf (robot description, URDF)
Before this commit: robot simple_quadruped, 5 links, 4 joints
Joints:
- joint hip_joint_bl: limit lower=-1.57 upper=1.57 effort=50 velocity=10 -> lower=-1.57 upper=1.57 effort=50 velocity=0.1
- joint hip_joint_br: limit lower=-1.57 upper=1.57 effort=50 velocity=10 -> lower=-1.57 upper=1.57 effort=50 velocity=0.1
- joint hip_joint_fl: limit lower=-1.57 upper=1.57 effort=50 velocity=10 -> lower=-1.57 upper=1.57 effort=50 velocity=0.1
- joint hip_joint_fr: limit lower=-1.57 upper=1.57 effort=50 velocity=10 -> lower=-1.57 upper=1.57 effort=50 velocity=0.1
